File: MCB1.sch (KiCad schematic (older format))
At the start: 34 parts, among them J1 SYNC, J10 Conn_01x12, J2 MIDI_OUT, J3 MIDI_IN, J4 MIDI_OUT, J5 MIDI_OUT, J6 TAPE_IN, J7 TAPE_OUT, J8 METRONOME, U1 74LS05, U3 H11L3

Commit message: WIP
Parts:
- D1: footprint Diode_THT:D_DO-35_SOD27_P7.62mm_Horizontal -> Diode_THT:D_DO-35_SOD27_P3.81mm_Vertical_AnodeUp
Changed lines of the file:
@@
 F 0 "D1" V 2004 1430 50  0000 L CNN
 F 1 "1N4148" H 1925 1225 50  0000 L CNN
-F 2 "Diode_THT:D_DO-35_SOD27_P7.62mm_Horizontal" H 2050 1175 50  0001 C CNN
+F 2 "Diode_THT:D_DO-35_SOD27_P3.81mm_Vertical_AnodeUp" H 2050 1175 50  0001 C CNN
 F 3 "https://assets.nexperia.com/documents/data-sheet/1N4148_1N4448.pdf" H 2050 1350 50  0001 C CNN
 	1    2050 1350
