File: MCB1.kicad_pcb (KiCad board)
At the start: 2 copper layers, 195.6 x 35.6 mm, 34 parts, among them J1 SYNC, J10 Conn_01x12, J2 MIDI_OUT, J3 MIDI_IN, J4 MIDI_OUT, J5 MIDI_OUT, J6 TAPE_IN, J7 TAPE_OUT, J8 METRONOME, U1 74LS05, U3 H11L3

Commit message: This board is worth building to test
Parts:
- moved J10 8.58 mm to (146.1, 100.5)
Routing:
- net /MIDI_RX: track 112.0 -> 2.79 mm, vias 1 -> 0
- net /METRONOME: track 68.5 -> 79.5 mm
- net /TAPE_IN: track 27.0 -> 35.8 mm
- net /CLOCK: track 39.0 -> 31.8 mm
- net /START: track 25.6 -> 18.3 mm
- net /CONTINUE: track 28.9 -> 21.7 mm
- net /TAPE_OUT: track 48.0 -> 53.7 mm
- net +5V: track 172.0 -> 176.5 mm
- net /MIDI_TX: track 38.8 -> 35.0 mm
- net GND: vias 75 -> 58
